File: 1.0/MiniVan.kicad_pcb (KiCad board)
At the start: 2 copper layers, 214 parts, among them J1 Reset Switch - A, J2 Reset Switch - B, J3 Reset Switch - C, U1 Elite-C - A, U2 Elite-C - B, U3 Elite-C - C

Commit message: 4/28/20 v4
Parts:
- added D105: D_Small, Diode_THT:D_DO-35_SOD27_P3.81mm_Vertical_AnodeUp, F.Cu at (140.5, 2.38)
- added D106: D_Small, Diode_THT:D_DO-35_SOD27_P3.81mm_Vertical_AnodeUp, F.Cu at (144.5, 2.38)
- added D107: D_Small, Diode_THT:D_DO-35_SOD27_P3.81mm_Vertical_AnodeUp, F.Cu at (132.6, 2.38)
- added D108: D_Small, Diode_THT:D_DO-35_SOD27_P3.81mm_Vertical_AnodeUp, F.Cu at (136.5, 2.38)
- added D109: D_Small, Diode_THT:D_DO-35_SOD27_P3.81mm_Vertical_AnodeUp, F.Cu at (149.2, 2.38)
- added D110: D_Small, Diode_THT:D_DO-35_SOD27_P3.81mm_Vertical_AnodeUp, F.Cu at (124.6, 2.38)
- added D111: D_Small, Diode_THT:D_DO-35_SOD27_P3.81mm_Vertical_AnodeUp, F.Cu at (128.6, 2.38)
- added D112: D_Small, Diode_THT:D_DO-35_SOD27_P3.81mm_Vertical_AnodeUp, F.Cu at (120.7, 2.38)
- added D113: D_Small, Diode_THT:D_DO-35_SOD27_P3.81mm_Vertical_AnodeUp, F.Cu at (146.8, -3.17)
- added D114: D_Small, Diode_THT:D_DO-35_SOD27_P3.81mm_Vertical_AnodeUp, F.Cu at (142.9, -3.17)
- added D115: D_Small, Diode_THT:D_DO-35_SOD27_P3.81mm_Vertical_AnodeUp, F.Cu at (134.9, -3.17)
- added D116: D_Small, Diode_THT:D_DO-35_SOD27_P3.81mm_Vertical_AnodeUp, F.Cu at (138.9, -3.17)
- added D117: D_Small, Diode_THT:D_DO-35_SOD27_P3.81mm_Vertical_AnodeUp, F.Cu at (131.0, -3.17)
- added D118: D_Small, Diode_THT:D_DO-35_SOD27_P3.81mm_Vertical_AnodeUp, F.Cu at (123.0, -3.17)
- added D119: D_Small, Diode_THT:D_DO-35_SOD27_P3.81mm_Vertical_AnodeUp, F.Cu at (127.0, -3.17)
- added D120: D_Small, Diode_THT:D_DO-35_SOD27_P3.81mm_Vertical_AnodeUp, F.Cu at (150.8, -3.17)
- added MX105: MX-NoLED, MX_Alps_Hybrid:MX-1U-NoLED, F.Cu at (-139.7, -0.79)
- added MX106: MX-NoLED, MX_Alps_Hybrid:MX-1U-NoLED, F.Cu at (-158.8, -0.79)
- added MX107: MX-NoLED, MX_Alps_Hybrid:MX-1U-NoLED, F.Cu at (-101.6, -0.79)
- added MX108: MX-NoLED, MX_Alps_Hybrid:MX-1U-NoLED, F.Cu at (-120.7, -0.79)
- added MX109: MX-NoLED, MX_Alps_Hybrid:MX-1U-NoLED, F.Cu at (-177.8, -0.79)
- added MX110: MX-NoLED, MX_Alps_Hybrid:MX-1U-NoLED, F.Cu at (-63.5, -0.79)
- added MX111: MX-NoLED, MX_Alps_Hybrid:MX-1U-NoLED, F.Cu at (-82.5, -0.79)
- added MX112: MX-NoLED, MX_Alps_Hybrid:MX-1U-NoLED, F.Cu at (-44.5, -0.79)
- added MX113: MX-NoLED, MX_Alps_Hybrid:MX-1U-NoLED, F.Cu at (-6.35, -0.79)
- added MX114: MX-NoLED, MX_Alps_Hybrid:MX-1U-NoLED, F.Cu at (12.7, -0.79)
- added MX115: MX-NoLED, MX_Alps_Hybrid:MX-1U-NoLED, F.Cu at (50.8, -0.79)
- added MX116: MX-NoLED, MX_Alps_Hybrid:MX-1U-NoLED, F.Cu at (31.8, -0.79)
- added MX117: MX-NoLED, MX_Alps_Hybrid:MX-1U-NoLED, F.Cu at (69.8, -0.79)
- added MX118: MX-NoLED, MX_Alps_Hybrid:MX-1U-NoLED, F.Cu at (108.0, -0.79)
- added MX119: MX-NoLED, MX_Alps_Hybrid:MX-1U-NoLED, F.Cu at (88.9, -0.79)
- added MX120: MX-NoLED, MX_Alps_Hybrid:MX-1U-NoLED, F.Cu at (-25.4, -0.79)
- U1, U2, U3: footprint Keebio-Parts:Elite-C-castellated-29pin -> Keebio-Parts:Elite-C-castellated-29pin-holes
- moved MX46 1456.9 mm to (1031.9, 211.9)
- moved MX33 1432.8 mm to (993.8, 211.9)
- moved MX27 1344.9 mm to (974.7, 211.9)
- moved MX7 1339.9 mm to (917.6, 211.9)
- moved MX51 1315.4 mm to (898.5, 211.9)
- moved MX39 1235.3 mm to (860.4, 211.9)
- moved MX32 1229.6 mm to (841.4, 211.9)
- moved MX45 1200.8 mm to (879.5, 211.9)
- moved MX13 1163.6 mm to (784.2, 211.9)
- moved MX52 844.9 mm to (1050.9, 211.9)
- moved D6 811.1 mm to (1099.3, 216.7), turned to 135 degrees
- moved D33 791.9 mm to (1080.3, 210.3), turned to 135 degrees
- moved D27 789.5 mm to (1085.1, 210.3), turned to 135 degrees
- moved D39 788.1 mm to (1075.5, 216.7), turned to 135 degrees
- moved D20 784.5 mm to (1089.8, 216.7), turned to 135 degrees
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Connections:
- D13 pad 1: row-A0 -> Net-(D13-Pad1)
- D14 pad 1: row-A1 -> Net-(D14-Pad1)
- D20 pad 1: row-A0 -> Net-(D13-Pad1)
- D21 pad 1: row-A1 -> Net-(D14-Pad1)
- D26 pad 1: row-A0 -> Net-(D13-Pad1)
- D27 pad 1: row-A1 -> Net-(D14-Pad1)
- D32 pad 1: row-A0 -> Net-(D13-Pad1)
- D33 pad 1: row-A1 -> Net-(D14-Pad1)
- D39 pad 1: row-A0 -> Net-(D13-Pad1)
- D40 pad 1: row-A1 -> Net-(D14-Pad1)
- D45 pad 1: row-A0 -> Net-(D13-Pad1)
- D46 pad 1: row-A1 -> Net-(D14-Pad1)
- D51 pad 1: row-A0 -> Net-(D13-Pad1)
- D52 pad 1: row-A1 -> Net-(D14-Pad1)
- D6 pad 1: row-A0 -> Net-(D13-Pad1)
- D7 pad 1: row-A1 -> Net-(D14-Pad1)
- MX13 pad 1: col-A1 -> Net-(MX13-Pad1)
- MX14 pad 1: col-A1 -> Net-(MX13-Pad1)
- MX20 pad 1: col-A2 -> Net-(MX20-Pad1)
- MX21 pad 1: col-A2 -> Net-(MX20-Pad1)
- MX26 pad 1: col-A3 -> Net-(MX26-Pad1)
- MX27 pad 1: col-A3 -> Net-(MX26-Pad1)
- MX32 pad 1: col-A4 -> Net-(MX32-Pad1)
- MX33 pad 1: col-A4 -> Net-(MX32-Pad1)
- MX38 pad 1: Net-(MX38-Pad1) -> col-C6
- MX39 pad 1: col-A5 -> Net-(MX39-Pad1)
- MX40 pad 1: col-A5 -> Net-(MX39-Pad1)
- MX45 pad 1: col-A6 -> Net-(MX45-Pad1)
- MX46 pad 1: col-A6 -> Net-(MX45-Pad1)
- MX51 pad 1: col-A7 -> Net-(MX51-Pad1)
- MX52 pad 1: col-A7 -> Net-(MX51-Pad1)
- MX6 pad 1: col-A0 -> Net-(MX6-Pad1)
- MX7 pad 1: col-A0 -> Net-(MX6-Pad1)
- U1 pad 10: Net-(U1-Pad10) -> row-A2
- U1 pad 11: row-A0 -> row-A3
- U1 pad 12: row-A1 -> row-A7
- U1 pad 13: col-A7 -> row-A0
- U1 pad 14: col-A6 -> row-A1
- U1 pad 15: col-A5 -> row-A6
- U1 pad 16: col-A4 -> row-A5
- U1 pad 17: col-A3 -> col-A0
- U1 pad 18: col-A2 -> Net-(U1-Pad18)
- U1 pad 19: col-A1 -> Net-(U1-Pad19)
- U1 pad 20: col-A0 -> Net-(U1-Pad20)
- U1 pad 8: Net-(U1-Pad8) -> col-A1
- U1 pad 9: Net-(U1-Pad9) -> row-A4
- U2 pad 10: row-B2 -> col-B4
- U2 pad 11: row-B3 -> col-B5
- U2 pad 12: row-B4 -> col-B6
- U2 pad 13: col-B6 -> row-B4
- U2 pad 14: col-B5 -> row-B3
- U2 pad 15: col-B4 -> row-B2
- U2 pad 16: col-B3 -> row-B1
- U2 pad 17: col-B2 -> row-B0
- U2 pad 18: col-B1 -> Net-(U2-Pad18)
- U2 pad 19: col-B0 -> Net-(U2-Pad19)
- U2 pad 5: Net-(U2-Pad5) -> col-B0
- U2 pad 6: Net-(U2-Pad6) -> col-B1
- U2 pad 7: Net-(U2-Pad7) -> col-B2
- U2 pad 8: row-B0 -> Net-(U2-Pad8)
- U2 pad 9: row-B1 -> col-B3
Routing:
- net Net-(D109-Pad2): track 0.00 -> 338.4 mm
- net col-A0: track 0.00 -> 328.5 mm, vias 0 -> 1
- net Net-(D106-Pad2): track 0.00 -> 315.2 mm
- net Net-(D105-Pad2): track 0.00 -> 290.3 mm
- net Net-(D91-Pad2): track 0.00 -> 278.1 mm
- net Net-(D108-Pad2): track 0.00 -> 267.2 mm
- net Net-(D90-Pad2): track 0.00 -> 245.7 mm
- net Net-(D107-Pad2): track 0.00 -> 242.9 mm
- net Net-(D94-Pad2): track 0.00 -> 229.7 mm
- net Net-(D111-Pad2): track 0.00 -> 219.4 mm
- net Net-(D96-Pad2): track 0.00 -> 198.8 mm
- net Net-(D110-Pad2): track 0.00 -> 196.1 mm
- net col-A1: track 0.00 -> 188.6 mm
- net col-B6: track 0.00 -> 180.1 mm
- net Net-(D120-Pad2): track 0.00 -> 177.2 mm
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- added copper zone on B.Cu, net gndB

Commit message: 4/30/20 v1
Parts:
- removed D13, D14, D20, D21, D26, D27, D32, D33, D39, D40, D45, D46, D51, D52, D6, D7: D_Small, Diode_THT:D_DO-35_SOD27_P3.81mm_Vertical_AnodeUp
- removed J1: Reset Switch - A, Connector_Wire:SolderWirePad_1x02_P3.81mm_Drill0.8mm
- removed J2: Reset Switch - B, Connector_Wire:SolderWirePad_1x02_P3.81mm_Drill0.8mm
- removed J3: Reset Switch - C, Connector_Wire:SolderWirePad_1x02_P3.81mm_Drill0.8mm
- removed MX13, MX14, MX20, MX21, MX26, MX27, MX32, MX33, MX39, MX40, MX45, MX46, MX51, MX52, MX6, MX7: MX-NoLED, MX_Alps_Hybrid:MX-1U-NoLED
- MX4: footprint MX_Alps_Hybrid:MX-2U-NoLED -> MX_Alps_Hybrid:MX-2.25U-NoLED
- moved MX8 817.3 mm to (-26.2, 73.0)
- moved D1 786.7 mm to (67.5, 50.0), turned to 315 degrees
- moved D11 781.9 mm to (77.0, 35.7), turned to 315 degrees
- moved MX9 771.3 mm to (-16.7, 92.1)
- moved D8 761.5 mm to (79.4, 50.0), turned to 315 degrees
- moved D10 760.1 mm to (77.8, 40.5), turned to 315 degrees
- moved D9 732.2 mm to (78.6, 45.2), turned to 315 degrees
- moved D31 730.4 mm to (112.7, 35.7), turned to 315 degrees
- moved MX11 729.2 mm to (-2.38, 130.2)
- moved D17 726.5 mm to (89.7, 40.5), turned to 315 degrees
- moved MX31 720.1 mm to (54.8, 130.2)
- moved D4 716.5 mm to (65.1, 35.7), turned to 315 degrees
- moved D36 710.1 mm to (125.4, 40.5), turned to 315 degrees
- moved D23 696.0 mm to (102.4, 45.2), turned to 315 degrees
- moved D16 693.4 mm to (90.5, 45.2), turned to 315 degrees
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Connections:
- U2 pad 10: col-B4 -> row-B2
- U2 pad 11: col-B5 -> row-B1
- U2 pad 12: col-B6 -> row-B0
- U2 pad 13: row-B4 -> col-B0
- U2 pad 14: row-B3 -> col-B1
- U2 pad 15: row-B2 -> col-B2
- U2 pad 16: row-B1 -> col-B3
- U2 pad 17: row-B0 -> col-B4
- U2 pad 18: Net-(U2-Pad18) -> col-B5
- U2 pad 19: Net-(U2-Pad19) -> col-B6
- U2 pad 5: col-B0 -> Net-(U2-Pad5)
- U2 pad 6: col-B1 -> Net-(U2-Pad6)
- U2 pad 7: col-B2 -> Net-(U2-Pad7)
- U2 pad 8: Net-(U2-Pad8) -> row-B4
- U2 pad 9: col-B3 -> row-B3
- U3 pad 10: col-C2 -> col-C5
- U3 pad 11: col-C1 -> col-C6
- U3 pad 12: col-C0 -> col-C7
- U3 pad 13: col-C10 -> col-C13
- U3 pad 14: col-C9 -> row-C0
- U3 pad 15: col-C8 -> row-C1
- U3 pad 16: col-C7 -> row-C2
- U3 pad 17: col-C6 -> row-C3
- U3 pad 18: col-C5 -> row-C4
- U3 pad 19: col-C4 -> Net-(U3-Pad19)
- U3 pad 20: col-C3 -> Net-(U3-Pad20)
- U3 pad 25: col-C13 -> col-C8
- U3 pad 26: col-C12 -> col-C9
- U3 pad 27: col-C11 -> col-C10
- U3 pad 28: Net-(U3-Pad28) -> col-C11
- U3 pad 29: Net-(U3-Pad29) -> col-C12
- U3 pad 5: row-C0 -> col-C0
- U3 pad 6: row-C1 -> col-C1
- U3 pad 7: row-C2 -> col-C2
- U3 pad 8: row-C3 -> col-C3
- U3 pad 9: row-C4 -> col-C4
Routing:
- net col-C13: track 0.00 -> 338.4 mm
- net col-C12: track 0.00 -> 303.6 mm
- net col-C11: track 0.00 -> 283.4 mm
- net col-C10: track 0.00 -> 272.8 mm
- net row-C4: track 0.00 -> 260.3 mm
- net row-C3: track 0.00 -> 259.9 mm
- net row-C2: track 0.00 -> 259.6 mm
- net row-C1: track 0.00 -> 259.4 mm
- net row-C0: track 0.00 -> 259.2 mm
- net Net-(D17-Pad2): track 0.00 -> 227.8 mm
- net col-C9: track 0.00 -> 224.8 mm
- net Net-(D5-Pad2): track 0.00 -> 223.7 mm
- net Net-(D65-Pad2): track 0.00 -> 219.5 mm
- net Net-(D12-Pad2): track 0.00 -> 219.5 mm
- net Net-(D19-Pad2): track 0.00 -> 215.6 mm
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- added copper zone on B.Cu, net gndA
- added copper zone on B.Cu, net gndC
Other:
- board outline added: 444.5 x 171.4 mm
- board text added: "40% Third row and the trunk"
- board text added: "60% The cabin and the middle row"
- board text added: "Detachable Luggage Rack"
- board text added: "The MiniVan"
- board text added: "rev1.0"

Commit message: 5/1/20 v1
Parts:
- moved D101 32.3 mm to (332.6, 17.5)
- moved D102 32.3 mm to (347.7, 36.5)
- moved D105 32.3 mm to (359.6, -4.76)
- moved D106 32.3 mm to (363.5, -4.76)
- moved D107 32.3 mm to (351.6, -4.76)
- moved D108 32.3 mm to (355.6, -4.76)
- moved D109 32.3 mm to (368.3, -4.76)
- moved D110 32.3 mm to (343.7, -4.76)
- moved D111 32.3 mm to (347.7, -4.76)
- moved D112 32.3 mm to (339.7, -4.76)
- moved D78 32.3 mm to (276.2, 36.5)
- moved D81 32.3 mm to (288.1, 36.5)
- moved D85 32.3 mm to (300.0, 36.5)
- moved D87 32.3 mm to (296.9, 17.5)
- moved D88 32.3 mm to (311.9, 36.5)
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Other:
- outline, holes or cut-outs redrawn
