File: 1.0/MiniVan.sch (KiCad schematic (older format))
At the start: 214 parts, among them J1 Reset Switch - A, J2 Reset Switch - B, J3 Reset Switch - C, U1 Elite-C - A, U2 Elite-C - B, U3 Elite-C - C

Commit message: 4/28/20 v4
Parts:
- added D105, D106, D107, D108, D109, D110, D111, D112, D113, D114, D115, D116, D117, D118, D119, D120: D_Small, Diode_THT:D_DO-35_SOD27_P3.81mm_Vertical_AnodeUp, symbol Device:D_Small
- added MX105, MX106, MX107, MX108, MX109, MX110, MX111, MX112, MX113, MX114, MX115, MX116, MX117, MX118, MX119, MX120: MX-NoLED, MX_Alps_Hybrid:MX-1U-NoLED, symbol MX_Alps_Hybrid:MX-NoLED
- U1, U2, U3: footprint Keebio-Parts:Elite-C-castellated-29pin -> Keebio-Parts:Elite-C-castellated-29pin-holes
Connections:
- net labels added: row-A2, row-A3, row-A4, row-A5, row-A6, row-A7
- net labels removed: col-A2, col-A3, col-A4, col-A5, col-A6, col-A7
- wire segments 207 -> 241
Other:
- moved on the sheet: D13, D14, D20, D21, D26, D27, D32, D33, D39, D40, D45, D46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

Commit message: 4/30/20 v1
Parts:
- removed D13, D14, D20, D21, D26, D27, D32, D33, D39, D40, D45, D46, D51, D52, D6, D7: D_Small, Diode_THT:D_DO-35_SOD27_P3.81mm_Vertical_AnodeUp, symbol Device:D_Small
- removed J1: Reset Switch - A, Connector_Wire:SolderWirePad_1x02_P3.81mm_Drill0.8mm, symbol Connector_Generic:Conn_02x01_Row_Letter_First
- removed J2: Reset Switch - B, Connector_Wire:SolderWirePad_1x02_P3.81mm_Drill0.8mm, symbol Connector_Generic:Conn_02x01_Row_Letter_First
- removed J3: Reset Switch - C, Connector_Wire:SolderWirePad_1x02_P3.81mm_Drill0.8mm, symbol Connector_Generic:Conn_02x01_Row_Letter_First
- removed MX13, MX14, MX20, MX21, MX26, MX27, MX32, MX33, MX39, MX40, MX45, MX46, MX51, MX52, MX6, MX7: MX-NoLED, MX_Alps_Hybrid:MX-1U-NoLED, symbol MX_Alps_Hybrid:MX-NoLED
- MX4: footprint MX_Alps_Hybrid:MX-2U-NoLED -> MX_Alps_Hybrid:MX-2.25U-NoLED
Connections:
- wire segments 241 -> 209

Commit message: 5/1/20 v1
Other:
- moved on the sheet: D1, D10, D100, D101, D102, D103, D104, D105, D106, D107, D108, D109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
